File: whistle-synth-v2/whistle-synth.kicad_pcb (KiCad board)
At the start: 2 copper layers, 99.5 x 85 mm, 138 parts, among them U1 LM358P

Commit message: check in
Parts:
- removed C1 (x6), C2 (x6), C4 (x6): 10uF, Capacitor_THT:CP_Radial_D4.0mm_P2.00mm
- removed C3 (x6): 4.7uF, Capacitor_THT:CP_Radial_D4.0mm_P2.00mm
- removed D1 (x6), D2 (x6): 1N5818, Diode_THT:D_DO-41_SOD81_P10.16mm_Horizontal
- removed H1 (x6): xlr3, MountingHole:MountingHole_2.2mm_M2_DIN965_Pad_TopBottom
- removed H2 (x6): xlr2, MountingHole:MountingHole_2.2mm_M2_DIN965_Pad_TopBottom
- removed H3 (x6): xlrG, MountingHole:MountingHole_2.2mm_M2_DIN965_Pad_TopBottom
- removed H4 (x6): Vo, MountingHole:MountingHole_2.2mm_M2_DIN965_Pad_TopBottom
- removed H5 (x6): gnd, MountingHole:MountingHole_2.2mm_M2_DIN965_Pad_TopBottom
- removed H6 (x6): 5v, MountingHole:MountingHole_2.2mm_M2_DIN965_Pad_TopBottom
- removed H7 (x6): 3.3v, MountingHole:MountingHole_2.2mm_M2_DIN965_Pad_TopBottom
- removed R1 (x6), R2 (x6), R7 (x6): 33R, Resistor_THT:R_Axial_DIN0309_L9.0mm_D3.2mm_P12.70mm_Horizontal
- removed R3 (x6), R5 (x6), R6 (x6): 10k, Resistor_THT:R_Axial_DIN0309_L9.0mm_D3.2mm_P12.70mm_Horizontal
- removed R4 (x6): 7.5R, Resistor_THT:R_Axial_DIN0309_L9.0mm_D3.2mm_P12.70mm_Horizontal
- removed REF** (x12): MountingHole_5mm, MountingHole:MountingHole_5mm
- removed U1 (x6): LM358P, Package_DIP:DIP-8_W7.62mm
Routing:
- net Net-(D1-A): track 296.2 -> 0.00 mm
- net Net-(U1A-+): track 200.7 -> 0.00 mm
- net Net-(D1-K): track 113.3 -> 0.00 mm
- net Net-(D2-K): track 108.9 -> 0.00 mm
- net Net-(C1-Pad1): track 95.2 -> 0.00 mm
- net Net-(U1A--): track 93.5 -> 0.00 mm
- net Net-(C2-Pad2): track 81.4 -> 0.00 mm
- net Net-(R3-Pad1): track 35.7 -> 0.00 mm
- net Net-(C2-Pad1): track 30.0 -> 0.00 mm
- net Net-(C1-Pad2): track 28.5 -> 0.00 mm
- net Net-(U1C-V+): track 26.5 -> 0.00 mm
- net Net-(C4-Pad2): track 24.0 -> 0.00 mm
- net Net-(H4-Pad1): track 21.0 -> 0.00 mm
Other:
- board outline removed
- board text removed: "Jeff Kaufman"
- board text removed: "Whistle Preamp v1"
